Commit message: migrated from bitbuket to github

File: src/arti_description/urdf/section_A_assembly.xacro (robot description, xacro)
@@ -4,5 +4,5 @@
     <model name='section_A_assembly'>
         <!-- Some Constants -->
-        <property name="PI" value="3.14159"/>
+        <xacro:property name="PI" value="3.14159"/>
         <!-- Wheel Properties -->
         <xacro:property name="wheel_length" value="0.03" />

File: src/arti_description/urdf/simple_car.xacro (robot description, xacro)
@@ -3,9 +3,9 @@
   <!-- Included URDF/XACRO Files -->
   <xacro:include filename="$(find arti_description)/urdf/arti_wheel_test.xacro" />
-  <property name="M_PI" value="3.14159"/>
+  <xacro:property name="M_PI" value="3.14159"/>
   <!-- Base Size -->
-  <property name="base_x_size" value="0.98740000" />
-  <property name="base_y_size" value="0.57090000" />
-  <property name="base_z_size" value="0.24750000" />
+  <xacro:property name="base_x_size" value="0.98740000" />
+  <xacro:property name="base_y_size" value="0.57090000" />
+  <xacro:property name="base_z_size" value="0.24750000" />
   <!-- Wheel Mounting Positions -->
   <xacro:property name="wheelbase" value="0.5120" />
